File: sclift_esp.sch (EAGLE design)
At the start: 18 parts, among them IC1 7805T

Commit message: Add files via upload
Parts:
- removed IC1: 7805T, linear:7805T
- added U$1: LM3940, lm3940:LM3940
Connections:
- net 3V3: now also U$1.VO; no longer IC1.VO
- net 5V: now also JP1.1, U$1.VI; no longer IC1.VI, JP2.2
- net GND: now also JP2.2, U$1.GND; no longer IC1.GND, JP1.1
Other:
- note removed: "*LM3940"
Changed lines of the file:
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@@
 <setting verticaltext="up"/>
 </settings>
-<grid distance="0.1" unitdist="inch" unit="inch" style="lines" multiple="1" display="no" altdistance="0.01" altunitdist="inch" altunit="inch"/>
+<grid distance="0.01" unitdist="inch" unit="inch" style="lines" multiple="1" display="no" altdistance="0.01" altunitdist="inch" altunit="inch"/>
 <layers>
 <layer number="1" name="Top" color="12" fill="1" visible="no" active="no"/>
@@
 <part name="C1" library="rcl" deviceset="C-EU" device="025-024X044"/>
 <part name="C2" library="rcl" deviceset="C-EU" device="025-024X044"/>
-<part name="IC1" library="linear" deviceset="78*" device="T" technology="05"/>
 <part name="GND1" library="supply1" deviceset="GND" device=""/>
 <part name="S1" library="switch-omron" deviceset="10-XX" device=""/>
@@
 <part name="JP2" library="pinhead" deviceset="PINHD-1X2" device=""/>
 <part name="R4" library="resistor" deviceset="R-US_" device="0204/7" value="10 kΩ"/>
+<part name="U$1" library="lm3940" deviceset="LM3940" device=""/>
 </parts>
 <sheets>
@@
 <sheet>
 <plain>
-<text x="52.578" y="54.102" size="1.27" layer="91">*LM3940</text>
 </plain>
 <instances>
 <instance part="C1" gate="G$1" x="32.258" y="46.482"/>
 <instance part="C2" gate="G$1" x="62.738" y="46.482"/>
-<instance part="IC1" gate="A1" x="47.498" y="49.022"/>
 <instance part="GND1" gate="1" x="47.498" y="36.322"/>
-<instance part="JP1" gate="G$1" x="50.292" y="69.85" rot="R180"/>
-<instance part="GND2" gate="1" x="59.944" y="62.484"/>
-<instance part="JP2" gate="G$1" x="41.91" y="69.85" rot="R180"/>
+<instance part="JP1" gate="G$1" x="9.398" y="42.164" rot="R180"/>
+<instance part="GND2" gate="1" x="3.556" y="32.766"/>
+<instance part="JP2" gate="G$1" x="1.016" y="42.164" rot="R180"/>
+<instance part="U$1" gate="G$1" x="47.498" y="49.022"/>
 </instances>
 <busses>
@@
 <segment>
 <pinref part="C1" gate="G$1" pin="2"/>
-<pinref part="IC1" gate="A1" pin="GND"/>
 <wire x1="32.258" y1="41.402" x2="47.498" y2="41.402" width="0.1524" layer="91"/>
 <pinref part="C2" gate="G$1" pin="2"/>
@@
 <wire x1="47.498" y1="41.402" x2="47.498" y2="38.862" width="0.1524" layer="91"/>
 <pinref part="GND1" gate="1" pin="GND"/>
-</segment>
-<segment>
-<pinref part="JP1" gate="G$1" pin="1"/>
-<wire x1="52.832" y1="67.31" x2="59.944" y2="67.31" width="0.1524" layer="91"/>
+<pinref part="U$1" gate="G$1" pin="GND"/>
+<junction x="47.498" y="41.402"/>
+</segment>
+<segment>
+<pinref part="JP2" gate="G$1" pin="2"/>
+<pinref part="JP2" gate="G$1" pin="1"/>
+<wire x1="3.556" y1="42.164" x2="3.556" y2="39.624" width="0.1524" layer="91"/>
+<wire x1="3.556" y1="39.624" x2="3.556" y2="35.306" width="0.1524" layer="91"/>
 <pinref part="GND2" gate="1" pin="GND"/>
-<wire x1="59.944" y1="65.024" x2="59.944" y2="67.31" width="0.1524" layer="91"/>
-<pinref part="JP2" gate="G$1" pin="1"/>
-<wire x1="44.45" y1="67.31" x2="52.832" y2="67.31" width="0.1524" layer="91"/>
 </segment>
 </net>
 <net name="3V3" class="0">
 <segment>
-<pinref part="IC1" gate="A1" pin="VO"/>
 <pinref part="C2" gate="G$1" pin="1"/>
 <wire x1="57.658" y1="49.022" x2="62.738" y2="49.022" width="0.1524" layer="91"/>
 <label x="62.738" y="49.022" size="1.27" layer="95" xref="yes"/>
+<pinref part="U$1" gate="G$1" pin="VO"/>
 </segment>
 </net>
@@
 <segment>
 <pinref part="C1" gate="G$1" pin="1"/>
-<pinref part="IC1" gate="A1" pin="VI"/>
 <wire x1="32.258" y1="49.022" x2="37.338" y2="49.022" width="0.1524" layer="91"/>
 <label x="32.258" y="49.022" size="1.27" layer="95" rot="R180" xref="yes"/>
-</segment>
-<segment>
+<pinref part="U$1" gate="G$1" pin="VI"/>
+</segment>
+<segment>
+<pinref part="JP1" gate="G$1" pin="1"/>
 <pinref part="JP1" gate="G$1" pin="2"/>
-<wire x1="52.832" y1="69.85" x2="60.706" y2="69.85" width="0.1524" layer="91"/>
-<label x="60.706" y="69.85" size="1.27" layer="95" xref="yes"/>
-<pinref part="JP2" gate="G$1" pin="2"/>
-<wire x1="52.832" y1="69.85" x2="44.45" y2="69.85" width="0.1524" layer="91"/>
+<wire x1="11.938" y1="39.624" x2="11.938" y2="42.164" width="0.1524" layer="91"/>
+<wire x1="11.938" y1="42.164" x2="11.938" y2="46.482" width="0.1524" layer="91"/>
+<label x="11.938" y="46.482" size="1.27" layer="95" rot="R90" xref="yes"/>
 </segment>
 </net>
 </nets>
 </sheet>
-<sheet>
-<plain>
-</plain>
-<instances>
-</instances>
-<busses>
-</busses>
-<nets>
-</nets>
-</sheet>
